File: lander_hardware/i2c.sch (KiCad schematic (older format))
At the start: 5 parts, among them J2 I2C Output, U4 bmp180

Commit message: Started associating footprints
Parts:
- U4: footprint (none) -> footprints:bmp180
Changed lines of the file:
@@
 F 0 "U4" H 3500 4150 60  0000 C CNN
 F 1 "bmp180" H 3850 3600 60  0000 C CNN
-F 2 "" H 3500 4150 60  0001 C CNN
+F 2 "footprints:bmp180" H 3500 4150 60  0001 C CNN
 F 3 "" H 3500 4150 60  0001 C CNN
 	1    3850 3600

Commit message: Board layout
Parts:
- removed J2: I2C Output, symbol Screw_Terminal_1x02
- added P9: I2C Out, Pin_Headers:Pin_Header_Straight_1x02_Pitch2.54mm, symbol CONN_01X02
- C8: footprint (none) -> Capacitors_THT:C_Disc_D10.0mm_W2.5mm_P5.00mm
- R7, R8: footprint (none) -> Resistors_THT:R_Axial_DIN0207_L6.3mm_D2.5mm_P10.16mm_Horizontal
Connections:
- net SCL: now also P9.2 (P2)
- net SDA: now also P9.1 (P1)
Changed lines of the file:
@@
 SDA
 $Comp
-L +3.3V #PWR025
+L +3.3V #PWR026
 U 1 1 58B6245A
 P 2550 2000
-F 0 "#PWR025" H 2550 1850 50  0001 C CNN
+F 0 "#PWR026" H 2550 1850 50  0001 C CNN
 F 1 "+3.3V" H 2550 2140 50  0000 C CNN
 F 2 "" H 2550 2000 50  0000 C CNN
@@
 $EndComp
 $Comp
-L GND #PWR026
+L GND #PWR027
 U 1 1 58B62470
 P 2550 2350
-F 0 "#PWR026" H 2550 2100 50  0001 C CNN
+F 0 "#PWR027" H 2550 2100 50  0001 C CNN
 F 1 "GND" H 2550 2200 50  0000 C CNN
 F 2 "" H 2550 2350 50  0000 C CNN
@@
 $EndComp
 $Comp
-L GND #PWR027
+L GND #PWR028
 U 1 1 58B625B6
 P 4000 2950
-F 0 "#PWR027" H 4000 2700 50  0001 C CNN
+F 0 "#PWR028" H 4000 2700 50  0001 C CNN
 F 1 "GND" H 4000 2800 50  0000 C CNN
 F 2 "" H 4000 2950 50  0000 C CNN
@@
 F 0 "C8" H 3075 4100 50  0000 L CNN
 F 1 "100nF" H 3075 3900 50  0000 L CNN
-F 2 "" H 3088 3850 50  0001 C CNN
+F 2 "Capacitors_THT:C_Disc_D10.0mm_W2.5mm_P5.00mm" H 3088 3850 50  0001 C CNN
 F 3 "" H 3050 4000 50  0000 C CNN
 	1    3050 4000
@@
 $EndComp
 $Comp
-L GND #PWR028
+L GND #PWR029
 U 1 1 58B62730
 P 3050 4250
-F 0 "#PWR028" H 3050 4000 50  0001 C CNN
+F 0 "#PWR029" H 3050 4000 50  0001 C CNN
 F 1 "GND" H 3050 4100 50  0000 C CNN
 F 2 "" H 3050 4250 50  0000 C CNN
@@
 $EndComp
 $Comp
-L +3.3V #PWR029
+L +3.3V #PWR030
 U 1 1 58B62748
 P 2850 3600
-F 0 "#PWR029" H 2850 3450 50  0001 C CNN
+F 0 "#PWR030" H 2850 3450 50  0001 C CNN
 F 1 "+3.3V" H 2850 3740 50  0000 C CNN
 F 2 "" H 2850 3600 50  0000 C CNN
@@
 $EndComp
 $Comp
-L +3.3V #PWR030
+L +3.3V #PWR031
 U 1 1 58B627A2
 P 4600 3050
-F 0 "#PWR030" H 4600 2900 50  0001 C CNN
+F 0 "#PWR031" H 4600 2900 50  0001 C CNN
 F 1 "+3.3V" H 4600 3190 50  0000 C CNN
 F 2 "" H 4600 3050 50  0000 C CNN
@@
 F 0 "R7" V 4680 3250 50  0000 C CNN
 F 1 "4.7K" V 4600 3250 50  0000 C CNN
-F 2 "" V 4530 3250 50  0001 C CNN
+F 2 "Resistors_THT:R_Axial_DIN0207_L6.3mm_D2.5mm_P10.16mm_Horizontal" V 4530 3250 50  0001 C CNN
 F 3 "" H 4600 3250 50  0000 C CNN
 	1    4600 3250
@@
 F 0 "R8" V 5130 3350 50  0000 C CNN
 F 1 "4.7K" V 5050 3350 50  0000 C CNN
-F 2 "" V 4980 3350 50  0001 C CNN
+F 2 "Resistors_THT:R_Axial_DIN0207_L6.3mm_D2.5mm_P10.16mm_Horizontal" V 4980 3350 50  0001 C CNN
 F 3 "" H 5050 3350 50  0000 C CNN
 	1    5050 3350
@@
 	5050 3500 5050 3600
 Connection ~ 5050 3600
-$Comp
-L Screw_Terminal_1x02 J2
-U 1 1 58B6EEC5
-P 5200 4150
-F 0 "J2" H 5200 4400 50  0000 C TNN
-F 1 "I2C Output" V 5050 4150 50  0000 C TNN
-F 2 "" H 5200 3925 50  0001 C CNN
-F 3 "" H 5175 4150 50  0001 C CNN
-	1    5200 4150
-	-1   0    0    -1
-$EndComp
 Wire Wire Line
 	4600 3400 4600 4050
@@
 	4750 4250 5000 4250
 Connection ~ 4750 3600
+$Comp
+L CONN_01X02 P9
+U 1 1 58BCBB20
+P 5250 4150
+F 0 "P9" H 5250 4300 50  0000 C CNN
+F 1 "I2C Out" V 5350 4150 50  0000 C CNN
+F 2 "Pin_Headers:Pin_Header_Straight_1x02_Pitch2.54mm" H 5250 4150 50  0001 C CNN
+F 3 "" H 5250 4150 50  0000 C CNN
+	1    5250 4150
+	1    0    0    -1
+$EndComp
+Wire Wire Line
+	5000 4050 5000 4100
+Wire Wire Line
+	5000 4100 5050 4100
+Wire Wire Line
+	5050 4200 5000 4200
+Wire Wire Line
+	5000 4200 5000 4250
 $EndSCHEMATC
