File: lander_hardware/pyro.sch (KiCad schematic (older format))
At the start: 14 parts, among them J3 Pyro Channel, J4 Pyro Channel, J5 Pyro Channel, P7 Continuity Jumpers, P8 Pyro Jumpers, Q1 Q_NPN_CBE, Q2 Q_NPN_CBE, Q3 Q_NPN_CBE

Commit message: Board layout
Parts:
- J3, J4, J5: footprint (none) -> Connectors:bornier2
- P7, P8: footprint (none) -> Pin_Headers:Pin_Header_Straight_2x03_Pitch2.54mm
- R10, R11, R12, R13, R14, R9: footprint (none) -> Resistors_THT:R_Axial_DIN0207_L6.3mm_D2.5mm_P10.16mm_Horizontal
Changed lines of the file:
@@
 F 0 "R9" V 2630 2500 50  0000 C CNN
 F 1 "1M" V 2550 2500 50  0000 C CNN
-F 2 "" V 2480 2500 50  0001 C CNN
+F 2 "Resistors_THT:R_Axial_DIN0207_L6.3mm_D2.5mm_P10.16mm_Horizontal" V 2480 2500 50  0001 C CNN
 F 3 "" H 2550 2500 50  0000 C CNN
 	1    2550 2500
@@
 F 0 "R11" V 5530 2500 50  0000 C CNN
 F 1 "1M" V 5450 2500 50  0000 C CNN
-F 2 "" V 5380 2500 50  0001 C CNN
+F 2 "Resistors_THT:R_Axial_DIN0207_L6.3mm_D2.5mm_P10.16mm_Horizontal" V 5380 2500 50  0001 C CNN
 F 3 "" H 5450 2500 50  0000 C CNN
 	1    5450 2500
@@
 F 0 "R13" V 8380 2500 50  0000 C CNN
 F 1 "1M" V 8300 2500 50  0000 C CNN
-F 2 "" V 8230 2500 50  0001 C CNN
+F 2 "Resistors_THT:R_Axial_DIN0207_L6.3mm_D2.5mm_P10.16mm_Horizontal" V 8230 2500 50  0001 C CNN
 F 3 "" H 8300 2500 50  0000 C CNN
 	1    8300 2500
@@
 $EndComp
 $Comp
-L GND #PWR031
+L GND #PWR032
 U 1 1 58A5FED3
 P 2300 2850
-F 0 "#PWR031" H 2300 2600 50  0001 C CNN
+F 0 "#PWR032" H 2300 2600 50  0001 C CNN
 F 1 "GND" H 2300 2700 50  0000 C CNN
 F 2 "" H 2300 2850 50  0000 C CNN
@@
 $EndComp
 $Comp
-L GND #PWR032
+L GND #PWR033
 U 1 1 58A5FEF9
 P 5200 2900
-F 0 "#PWR032" H 5200 2650 50  0001 C CNN
+F 0 "#PWR033" H 5200 2650 50  0001 C CNN
 F 1 "GND" H 5200 2750 50  0000 C CNN
 F 2 "" H 5200 2900 50  0000 C CNN
@@
 $EndComp
 $Comp
-L GND #PWR033
+L GND #PWR034
 U 1 1 58A5FFD3
 P 8050 2900
-F 0 "#PWR033" H 8050 2650 50  0001 C CNN
+F 0 "#PWR034" H 8050 2650 50  0001 C CNN
 F 1 "GND" H 8050 2750 50  0000 C CNN
 F 2 "" H 8050 2900 50  0000 C CNN
@@
 $EndComp
 $Comp
-L +6V #PWR034
+L +6V #PWR035
 U 1 1 58A6013C
 P 2750 2000
-F 0 "#PWR034" H 2750 1850 50  0001 C CNN
+F 0 "#PWR035" H 2750 1850 50  0001 C CNN
 F 1 "+6V" H 2750 2140 50  0000 C CNN
 F 2 "" H 2750 2000 50  0000 C CNN
@@
 $EndComp
 $Comp
-L +6V #PWR035
+L +6V #PWR036
 U 1 1 58A60162
 P 5700 2000
-F 0 "#PWR035" H 5700 1850 50  0001 C CNN
+F 0 "#PWR036" H 5700 1850 50  0001 C CNN
 F 1 "+6V" H 5700 2140 50  0000 C CNN
 F 2 "" H 5700 2000 50  0000 C CNN
@@
 $EndComp
 $Comp
-L +6V #PWR036
+L +6V #PWR037
 U 1 1 58A60188
 P 8550 2050
-F 0 "#PWR036" H 8550 1900 50  0001 C CNN
+F 0 "#PWR037" H 8550 1900 50  0001 C CNN
 F 1 "+6V" H 8550 2190 50  0000 C CNN
 F 2 "" H 8550 2050 50  0000 C CNN
@@
 F 0 "P7" H 4650 5050 50  0000 C CNN
 F 1 "Continuity Jumpers" H 4650 4650 50  0000 C CNN
-F 2 "" H 4650 3650 50  0001 C CNN
+F 2 "Pin_Headers:Pin_Header_Straight_2x03_Pitch2.54mm" H 4650 3650 50  0001 C CNN
 F 3 "" H 4650 3650 50  0000 C CNN
 	1    4650 4850
@@
 F 0 "R10" V 2980 3700 50  0000 C CNN
 F 1 "100K" V 2900 3700 50  0000 C CNN
-F 2 "" V 2830 3700 50  0001 C CNN
+F 2 "Resistors_THT:R_Axial_DIN0207_L6.3mm_D2.5mm_P10.16mm_Horizontal" V 2830 3700 50  0001 C CNN
 F 3 "" H 2900 3700 50  0000 C CNN
 	1    2900 3700
@@
 F 0 "R12" V 5730 3700 50  0000 C CNN
 F 1 "100K" V 5650 3700 50  0000 C CNN
-F 2 "" V 5580 3700 50  0001 C CNN
+F 2 "Resistors_THT:R_Axial_DIN0207_L6.3mm_D2.5mm_P10.16mm_Horizontal" V 5580 3700 50  0001 C CNN
 F 3 "" H 5650 3700 50  0000 C CNN
 	1    5650 3700
@@
 F 0 "R14" V 8480 3700 50  0000 C CNN
 F 1 "100K" V 8400 3700 50  0000 C CNN
-F 2 "" V 8330 3700 50  0001 C CNN
+F 2 "Resistors_THT:R_Axial_DIN0207_L6.3mm_D2.5mm_P10.16mm_Horizontal" V 8330 3700 50  0001 C CNN
 F 3 "" H 8400 3700 50  0000 C CNN
 	1    8400 3700
@@
 F 0 "P8" H 4700 1400 50  0000 C CNN
 F 1 "Pyro Jumpers" H 4700 1000 50  0000 C CNN
-F 2 "" H 4700 0   50  0001 C CNN
+F 2 "Pin_Headers:Pin_Header_Straight_2x03_Pitch2.54mm" H 4700 0   50  0001 C CNN
 F 3 "" H 4700 0   50  0000 C CNN
 	1    4700 1200
@@
 GNDin
 $Comp
-L +6V #PWR037
+L +6V #PWR038
 U 1 1 58B345BF
 P 1950 950
-F 0 "#PWR037" H 1950 800 50  0001 C CNN
+F 0 "#PWR038" H 1950 800 50  0001 C CNN
 F 1 "+6V" H 1950 1090 50  0000 C CNN
 F 2 "" H 1950 950 50  0000 C CNN
@@
 $EndComp
 $Comp
-L GND #PWR038
+L GND #PWR039
 U 1 1 58B34637
 P 1850 1200
-F 0 "#PWR038" H 1850 950 50  0001 C CNN
+F 0 "#PWR039" H 1850 950 50  0001 C CNN
 F 1 "GND" H 1850 1050 50  0000 C CNN
 F 2 "" H 1850 1200 50  0000 C CNN
@@
 F 0 "J3" H 2950 2450 50  0000 C TNN
 F 1 "Pyro Channel" V 2800 2200 50  0000 C TNN
-F 2 "" H 2950 1975 50  0001 C CNN
+F 2 "Connectors:bornier2" H 2950 1975 50  0001 C CNN
 F 3 "" H 2925 2200 50  0001 C CNN
 	1    2950 2200
@@
 F 0 "J4" H 5900 2450 50  0000 C TNN
 F 1 "Pyro Channel" V 5750 2200 50  0000 C TNN
-F 2 "" H 5900 1975 50  0001 C CNN
+F 2 "Connectors:bornier2" H 5900 1975 50  0001 C CNN
 F 3 "" H 5875 2200 50  0001 C CNN
 	1    5900 2200
@@
 F 0 "J5" H 8750 2450 50  0000 C TNN
 F 1 "Pyro Channel" V 8600 2200 50  0000 C TNN
-F 2 "" H 8750 1975 50  0001 C CNN
+F 2 "Connectors:bornier2" H 8750 1975 50  0001 C CNN
 F 3 "" H 8725 2200 50  0001 C CNN
 	1    8750 2200

Commit message: Fixed power transistors being CBE instead of BCE
Parts:
- removed Q1, Q2, Q3: Q_NPN_CBE, TO_SOT_Packages_THT:TO-220_Vertical, symbol Q_NPN_CBE
- added Q1, Q2, Q3: Q_NPN_BCE, TO_SOT_Packages_THT:TO-220_Vertical, symbol Q_NPN_BCE
Changed lines of the file:
@@
 $EndDescr
-$Comp
-L Q_NPN_CBE Q1
-U 1 1 58A5F01A
-P 1800 2500
-F 0 "Q1" H 2000 2550 50  0000 L CNN
-F 1 "Q_NPN_CBE" H 2000 2450 50  0000 L CNN
-F 2 "TO_SOT_Packages_THT:TO-220_Vertical" H 2000 2600 50  0001 C CNN
-F 3 "" H 1800 2500 50  0000 C CNN
-	1    1800 2500
-	1    0    0    -1
-$EndComp
-$Comp
-L Q_NPN_CBE Q2
-U 1 1 58A5F107
-P 4700 2500
-F 0 "Q2" H 4900 2550 50  0000 L CNN
-F 1 "Q_NPN_CBE" H 4900 2450 50  0000 L CNN
-F 2 "TO_SOT_Packages_THT:TO-220_Vertical" H 4900 2600 50  0001 C CNN
-F 3 "" H 4700 2500 50  0000 C CNN
-	1    4700 2500
-	1    0    0    -1
-$EndComp
-$Comp
-L Q_NPN_CBE Q3
-U 1 1 58A5F146
-P 7550 2500
-F 0 "Q3" H 7750 2550 50  0000 L CNN
-F 1 "Q_NPN_CBE" H 7750 2450 50  0000 L CNN
-F 2 "TO_SOT_Packages_THT:TO-220_Vertical" H 7750 2600 50  0001 C CNN
-F 3 "" H 7550 2500 50  0000 C CNN
-	1    7550 2500
-	1    0    0    -1
-$EndComp
 $Comp
 L R R9
@@
 Wire Wire Line
 	2750 3700 2050 3700
+$Comp
+L Q_NPN_BCE Q1
+U 1 1 58C079F0
+P 1800 2500
+F 0 "Q1" H 2000 2550 50  0000 L CNN
+F 1 "Q_NPN_BCE" H 2000 2450 50  0000 L CNN
+F 2 "TO_SOT_Packages_THT:TO-220_Vertical" H 2000 2600 50  0001 C CNN
+F 3 "" H 1800 2500 50  0000 C CNN
+	1    1800 2500
+	1    0    0    -1
+$EndComp
+$Comp
+L Q_NPN_BCE Q2
+U 1 1 58C07A2D
+P 4700 2500
+F 0 "Q2" H 4900 2550 50  0000 L CNN
+F 1 "Q_NPN_BCE" H 4900 2450 50  0000 L CNN
+F 2 "TO_SOT_Packages_THT:TO-220_Vertical" H 4900 2600 50  0001 C CNN
+F 3 "" H 4700 2500 50  0000 C CNN
+	1    4700 2500
+	1    0    0    -1
+$EndComp
+$Comp
+L Q_NPN_BCE Q3
+U 1 1 58C07A64
+P 7550 2500
+F 0 "Q3" H 7750 2550 50  0000 L CNN
+F 1 "Q_NPN_BCE" H 7750 2450 50  0000 L CNN
+F 2 "TO_SOT_Packages_THT:TO-220_Vertical" H 7750 2600 50  0001 C CNN
+F 3 "" H 7550 2500 50  0000 C CNN
+	1    7550 2500
+	1    0    0    -1
+$EndComp
 $EndSCHEMATC
